Commit message: Fix ramsis

File: src/quori_description/urdf/ramsis_kinematics.xacro (robot description, xacro)
@@ -41,5 +41,5 @@
   <link name="ramsis/turret_link">
   </link>
-  <link name="ramsis/left_wheel_link">
+  <link name="ramsis/l_wheel_link">
     <inertial>
       <origin xyz="0 0 0" rpy="0 0 0"/>
@@ -48,5 +48,5 @@
     </inertial>
   </link>
-  <link name="ramsis/right_wheel_link">
+  <link name="ramsis/r_wheel_link">
     <inertial>
       <origin xyz="0 0 0" rpy="0 0 0"/>
@@ -65,6 +65,6 @@
     <origin xyz="0 0.12284075 0" rpy="0 0 0"/>
     <parent link="ramsis/wheel_axle"/>
-    <child link="ramsis/left_wheel_link"/>
-    <axis xyz="0 0 1" />
+    <child link="ramsis/l_wheel_link"/>
+    <axis xyz="0 1 0" />
     <limit effort="1" velocity="0.5"/>
   </joint>
@@ -72,6 +72,6 @@
     <origin xyz="0 -0.12284075 0" rpy="0 0 0"/>
     <parent link="ramsis/wheel_axle"/>
-    <child link="ramsis/right_wheel_link"/>
-    <axis xyz="0 0 1" />
+    <child link="ramsis/r_wheel_link"/>
+    <axis xyz="0 1 0" />
     <limit effort="1" velocity="0.5"/>
   </joint>

Commit message: Add base_link_diff

File: src/quori_description/urdf/ramsis_kinematics.xacro (robot description, xacro)
@@ -7,5 +7,5 @@
     <color rgba="0.3 0.3 0.3 1"/>
   </material>
-  <link name="ramsis/base_link">
+  <link name="ramsis/base_link_diff">
     <inertial>
       <origin xyz="0 0 0.1013587" rpy="0 0 0"/>
@@ -36,8 +36,10 @@
   <joint name="laser_scanner_joint" type="fixed">
     <origin xyz="0.178 0 0.1" rpy="0 0 0" />
-    <parent link="ramsis/base_link" />
+    <parent link="ramsis/base_link_diff" />
     <child link="ramsis/base_laser_scanner" />
   </joint>
   <link name="ramsis/turret_link">
+  </link>
+  <link name="ramsis/base_link">
   </link>
   <link name="ramsis/l_wheel_link">
@@ -58,4 +60,9 @@
     <origin xyz="0.1 0 -0.075" />
     <parent link="ramsis/wheel_axle" />
+    <child link="ramsis/base_link_diff" />
+  </joint>
+  <joint name="turret2base" type="fixed">
+    <origin xyz="0 0 -0.2027174" />
+    <parent link="ramsis/turret_link" />
     <child link="ramsis/base_link" />
   </joint>

Commit message: Fix base_link

File: src/quori_description/urdf/ramsis_kinematics.xacro (robot description, xacro)
@@ -85,5 +85,5 @@
   <joint name="turret" type="continuous">
     <origin xyz="0 0 0.2027174" rpy="0 0 0"/>
-    <parent link="ramsis/base_link"/>
+    <parent link="ramsis/base_link_diff"/>
     <child link="ramsis/turret_link"/>
     <axis xyz="0 0 1" />

Commit message: updated the laser to match the physical model better. rm middle file so laser attached to the ramsis frame directly

File: src/quori_description/urdf/ramsis_kinematics.xacro (robot description, xacro)
@@ -35,5 +35,5 @@
   </link>
   <joint name="laser_scanner_joint" type="fixed">
-    <origin xyz="0.178 0 0.1" rpy="0 0 0" />
+    <origin xyz="0.152 0 0.156" rpy="0 0.0 -1.5707" />
     <parent link="ramsis/base_link_diff" />
     <child link="ramsis/base_laser_scanner" />
