Commit message: Eliminated errors, still need to fix invisible gazebo model

File: src/quori_description/urdf/quori.xacro (robot description, xacro)
@@ -5,4 +5,16 @@
   <quori_kinematics />
   <ramsis_kinematics />
+  <material name="blue">
+    <color rgba="0 0 0.8 1"/>
+  </material>
+  <material name="black">
+    <color rgba="0 0 0 1"/>
+  </material>
+  <material name="white">
+    <color rgba="1 1 1 1"/>
+  </material>
+  <material name="gray">
+    <color rgba="0.5 0.5 0.5 1"/>
+  </material>
   <!-- Join the quori robot to the ramsis robot's turret joint -->
   <joint name="ramsis_quori_connector" type="fixed">
@@ -10,3 +22,71 @@
     <child link="quori/base_link"/>
   </joint>
+  <link name="base_link"/>
+  <joint name="fixed" type="fixed">
+    <parent link="ramsis/base_link"/>
+    <child link="base_link"/>
+  </joint>
+  <xacro:macro name="joint_transmission" params="prefix">
+    <transmission name="${prefix}_tran">
+      <type>transmission_interface/SimpleTransmission</type>
+      <actuator name="${prefix}_motor">
+        <hardwareInterface>hardware_interface/PositionJointInterface</hardwareInterface>
+        <mechanicalReduction>1</mechanicalReduction>
+      </actuator>
+      <joint name="${prefix}">
+        <hardwareInterface>hardware_interface/PositionJointInterface</hardwareInterface>
+      </joint>
+    </transmission>
+  </xacro:macro>
+  <xacro:macro name="wheel_transmission" params="prefix">
+    <transmission name="${prefix}_tran">
+      <type>transmission_interface/SimpleTransmission</type>
+      <actuator name="${prefix}_motor">
+        <hardwareInterface>hardware_interface/VelocityJointInterface</hardwareInterface>
+        <mechanicalReduction>1</mechanicalReduction>
+      </actuator>
+      <joint name="${prefix}">
+        <hardwareInterface>hardware_interface/VelocityJointInterface</hardwareInterface>
+      </joint>
+    </transmission>
+  </xacro:macro>
+  <xacro:joint_transmission prefix="waist_pitch"/>
+  <xacro:joint_transmission prefix="r_shoulder_pitch"/>
+  <xacro:joint_transmission prefix="r_shoulder_roll"/>
+  <xacro:joint_transmission prefix="l_shoulder_pitch"/>
+  <xacro:joint_transmission prefix="l_shoulder_roll"/>
+  <xacro:wheel_transmission prefix="l_wheel"/>
+  <xacro:wheel_transmission prefix="r_wheel"/>
+  <xacro:joint_transmission prefix="turret"/>
+  <gazebo reference="quori/body_upper">
+    <material>Gazebo/White</material>
+  </gazebo>
+  <gazebo reference="quori/base_link">
+    <material>Gazebo/White</material>
+  </gazebo>
+  <gazebo reference="quori/head">
+    <material>Gazebo/White</material>
+  </gazebo>
+  <gazebo reference="quori/r_arm_upper">
+    <material>Gazebo/White</material>
+  </gazebo>
+  <gazebo reference="quori/r_arm_lower">
+    <material>Gazebo/White</material>
+  </gazebo>
+  <gazebo reference="quori/l_arm_upper">
+    <material>Gazebo/White</material>
+  </gazebo>
+  <gazebo reference="quori/l_arm_lower">
+    <material>Gazebo/White</material>
+  </gazebo>
+  <gazebo reference="base_link_diff">
+    <material>Gazebo/White</material>
+  </gazebo>
+  <gazebo>
+    <plugin name="gazebo_ros_control" filename="libgazebo_ros_control.so">
+      <robotNamespace>/quori</robotNamespace>
+      <robotSimType>gazebo_ros_control/DefaultRobotHWSim</robotSimType>
+      <legacyModeNS>true</legacyModeNS>
+    </plugin>
+  </gazebo>
 </robot>

File: src/quori_description/urdf/quori_kinematics.xacro (robot description, xacro)
@@ -37,6 +37,6 @@
     <inertial>
       <origin xyz="0 0 0" rpy="0 0 0"/>
-      <mass value="0.0"/>
-      <inertia ixx="0.0"  ixy="0"  ixz="0" iyy="0.0" iyz="0" izz="0.0" />
+      <mass value="0.01"/>
+      <inertia ixx="0.01"  ixy="0"  ixz="0" iyy="0.0" iyz="0" izz="0.0" />
     </inertial>
   </link>
@@ -51,6 +51,6 @@
     <inertial>
       <origin xyz="0 0 0" rpy="0 0 0"/>
-      <mass value="0.00"/>
-      <inertia ixx="0.0"  ixy="0"  ixz="0" iyy="0.0" iyz="0" izz="0.0" />
+      <mass value="0.01"/>
+      <inertia ixx="0.1"  ixy="0"  ixz="0" iyy="0.0" iyz="0" izz="0.0" />
     </inertial>
     <visual>
@@ -89,6 +89,6 @@
     <inertial>
       <origin xyz="0 0 0" rpy="0 0 0"/>
-      <mass value="0.00"/>
-      <inertia ixx="0.0"  ixy="0"  ixz="0" iyy="0.0" iyz="0" izz="0.0" />
+      <mass value="0.01"/>
+      <inertia ixx="0.1"  ixy="0"  ixz="0" iyy="0.0" iyz="0" izz="0.0" />
     </inertial>
     <visual>
@@ -107,6 +107,6 @@
     <inertial>
       <origin xyz="0 0 0" rpy="0 0 0"/>
-      <mass value="0.0"/>
-      <inertia ixx="0.0"  ixy="0"  ixz="0" iyy="0.0" iyz="0" izz="0.0" />
+      <mass value="0.1"/>
+      <inertia ixx="0.1"  ixy="0"  ixz="0" iyy="0.0" iyz="0" izz="0.0" />
     </inertial>
   </link>
@@ -121,6 +121,6 @@
     <inertial>
       <origin xyz="0 0 0" rpy="0 0 0" />
-      <mass value="0.00" />
-      <inertia ixx="0.0"  ixy="0"  ixz="0" iyy="0.0" iyz="0" izz="0.0" />
+      <mass value="0.01" />
+      <inertia ixx="0.1"  ixy="0"  ixz="0" iyy="0.0" iyz="0" izz="0.0" />
     </inertial>
     <visual>
@@ -159,6 +159,6 @@
     <inertial>
       <origin xyz="0 0 0" rpy="0 0 0"/>
-      <mass value="0.00"/>
-      <inertia ixx="0.0"  ixy="0"  ixz="0" iyy="0.0" iyz="0" izz="0.0" />
+      <mass value="0.01"/>
+      <inertia ixx="0.1"  ixy="0"  ixz="0" iyy="0.0" iyz="0" izz="0.0" />
     </inertial>
     <visual>
@@ -229,5 +229,5 @@
       <origin xyz="0 0 0" rpy="0 0 0"/>
       <mass value="0.05"/>
-      <inertia ixx="0.0"  ixy="0"  ixz="0" iyy="0.0" iyz="0" izz="0.0" />
+      <inertia ixx="0.1"  ixy="0"  ixz="0" iyy="0.0" iyz="0" izz="0.0" />
     </inertial>
     <visual>

File: src/quori_description/urdf/ramsis_kinematics.xacro (robot description, xacro)
@@ -40,12 +40,22 @@
   </joint>
   <link name="ramsis/turret_link">
+    <inertial>
+      <origin xyz="0 0 0" rpy="0 0 0"/>
+      <mass value="0.01"/>
+      <inertia ixx="0.01"  ixy="0"  ixz="0" iyy="0.0" iyz="0" izz="0.0" />
+    </inertial>
   </link>
   <link name="ramsis/base_link">
+    <inertial>
+      <origin xyz="0 0 0" rpy="0 0 0"/>
+      <mass value="0.01"/>
+      <inertia ixx="0.01"  ixy="0"  ixz="0" iyy="0.0" iyz="0" izz="0.0" />
+    </inertial>
   </link>
   <link name="ramsis/l_wheel_link">
     <inertial>
       <origin xyz="0 0 0" rpy="0 0 0"/>
-      <mass value="0.0"/>
-      <inertia ixx="0.0"  ixy="0"  ixz="0" iyy="0.0" iyz="0" izz="0.0" />
+      <mass value="0.1"/>
+      <inertia ixx="0.1"  ixy="0"  ixz="0" iyy="0.0" iyz="0" izz="0.0" />
     </inertial>
   </link>
@@ -53,6 +63,6 @@
     <inertial>
       <origin xyz="0 0 0" rpy="0 0 0"/>
-      <mass value="0.0"/>
-      <inertia ixx="0.0"  ixy="0"  ixz="0" iyy="0.0" iyz="0" izz="0.0" />
+      <mass value="0.1"/>
+      <inertia ixx="0.1"  ixy="0"  ixz="0" iyy="0.0" iyz="0" izz="0.0" />
     </inertial>
   </link>
@@ -68,4 +78,9 @@
   </joint>
   <link name="ramsis/wheel_axle">
+    <inertial>
+      <origin xyz="0 0 0" rpy="0 0 0"/>
+      <mass value="0.00"/>
+      <inertia ixx="0.00"  ixy="0"  ixz="0" iyy="0.0" iyz="0" izz="0.0" />
+    </inertial>
   </link>
   <joint name="l_wheel" type="continuous">

Commit message: Fixed Gazebo model not visible

File: src/quori_description/urdf/quori.xacro (robot description, xacro)
@@ -22,7 +22,7 @@
     <child link="quori/base_link"/>
   </joint>
-  <link name="base_link"/>
+  <link name="world"/>
   <joint name="fixed" type="fixed">
-    <parent link="base_link"/>
+    <parent link="world"/>
     <child link="ramsis/wheel_axle"/>
   </joint>
