Commit message: Change r1 joints to revolute with position limits

File: src/quori_description/urdf/quori_kinematics.xacro (robot description, xacro)
@@ -41,10 +41,10 @@
     </inertial>
   </link>
-  <joint name="right_arm_r1" type="continuous">
+  <joint name="right_arm_r1" type="revolute">
     <origin xyz="0.015 -0.16403066 0.43021758" rpy="0 0 0"/>
     <parent link="quori/upper_torso"/>
     <child link="quori/right_arm_base"/>
     <axis xyz="0 -1 0" />
-    <limit effort="1" velocity="1"/>
+    <limit lower="-2.4" upper="2.4" effort="1" velocity="1"/>
   </joint>
   <link name="quori/right_arm_upper">
@@ -113,10 +113,10 @@
     </inertial>
   </link>
-  <joint name="left_arm_r1" type="continuous">
+  <joint name="left_arm_r1" type="revolute">
     <origin xyz="0.015 0.16403066 0.43021758" rpy="0 0 0"/>
     <parent link="quori/upper_torso"/>
     <child link="quori/left_arm_base"/>
     <axis xyz="0 1 0" />
-    <limit effort="1" velocity="1"/>
+    <limit lower="-2.4" upper="2.4" effort="1" velocity="1"/>
   </joint>
   <link name="quori/left_arm_upper">

Commit message: Provisional fixes to quori_description

File: src/quori_description/urdf/quori_kinematics.xacro (robot description, xacro)
@@ -10,5 +10,5 @@
       <origin rpy="0 0 -1.57079632679" xyz="0.02 0 -0.2007174"/>
       <geometry>
-        <mesh filename="package://quori_description/meshes/180915_Lower Torso.dae"/>
+        <mesh filename="package://quori_description/meshes/180915_Lower_Torso.dae"/>
       </geometry>
     </visual>
@@ -23,5 +23,5 @@
       <origin rpy="0 0 -1.57079632679" xyz="0.02 0 -0.5476974"/>
       <geometry>
-        <mesh filename="package://quori_description/meshes/0917_Upper Torso+Waist.dae"/>
+        <mesh filename="package://quori_description/meshes/0917_Upper_Torso+Waist.dae"/>
       </geometry>
     </visual>
@@ -57,5 +57,5 @@
       <origin rpy="-1.57079632679 0 0" xyz="0.165 -0.9765 -0.137"/>
       <geometry>
-        <mesh filename="package://quori_description/meshes/0917_Upper Arm+gear_right.dae"/>
+        <mesh filename="package://quori_description/meshes/0917_Upper_Arm+gear_right.dae"/>
       </geometry>
     </visual>
@@ -129,5 +129,5 @@
       <origin rpy="-1.57079632679 0 -3.14" xyz="0.165 0.9765 -0.137"/>
       <geometry>
-        <mesh filename="package://quori_description/meshes/0917_Upper Arm+gear_left.dae"/>
+        <mesh filename="package://quori_description/meshes/0917_Upper_Arm+gear_left.dae"/>
       </geometry>
     </visual>
@@ -167,5 +167,5 @@
       <origin rpy="-1.57 3.14 0" xyz="0 0 0" />
       <geometry>
-        <mesh filename="package://quori_description/meshes/0917_Lower Arm_right.dae" />
+        <mesh filename="package://quori_description/meshes/0917_Lower_Arm_right.dae" />
       </geometry>
     </visual>

Commit message: Fix URDF

File: src/quori_description/urdf/quori_kinematics.xacro (robot description, xacro)
@@ -167,5 +167,5 @@
       <origin rpy="-1.57 3.14 0" xyz="0 0 0" />
       <geometry>
-        <mesh filename="package://quori_description/meshes/0917_Lower_Arm_right.dae" />
+        <mesh filename="package://quori_description/meshes/0917_Lower_Arm_left.dae" />
       </geometry>
     </visual>

Commit message: Beginning of URDF changes

File: src/quori_description/urdf/quori_kinematics.xacro (robot description, xacro)
@@ -27,5 +27,5 @@
     </visual>
   </link>
-  <joint name="waist_hinge" type="revolute">
+  <joint name="waist_pitch" type="revolute">
     <origin xyz="0 0 0.34798" rpy="0 0 0"/>
     <parent link="quori/base_link"/>
@@ -41,5 +41,5 @@
     </inertial>
   </link>
-  <joint name="right_arm_r1" type="revolute">
+  <joint name="r_shoulder_pitch" type="revolute">
     <origin xyz="0.015 -0.16403066 0.43021758" rpy="0 0 0"/>
     <parent link="quori/upper_torso"/>
@@ -61,5 +61,5 @@
     </visual>
   </link>
-  <joint name="right_arm_r2" type="revolute">
+  <joint name="r_shoulder_roll" type="revolute">
     <origin xyz="0 0 0" rpy="0 -1.57 0"/>
     <parent link="quori/right_arm_base"/>
@@ -113,5 +113,5 @@
     </inertial>
   </link>
-  <joint name="left_arm_r1" type="revolute">
+  <joint name="l_shoulder_pitch" type="revolute">
     <origin xyz="0.015 0.16403066 0.43021758" rpy="0 0 0"/>
     <parent link="quori/upper_torso"/>
@@ -133,5 +133,5 @@
     </visual>
   </link>
-  <joint name="left_arm_r2" type="revolute">
+  <joint name="l_shoulder_roll" type="revolute">
     <origin xyz="0 0 0" rpy="0 -1.57 0"/>
     <parent link="quori/left_arm_base"/>
@@ -198,5 +198,5 @@
     </visual>
   </link>
-  <joint name="head_joint" type="fixed">
+  <joint name="neck" type="fixed">
     <origin xyz="0 0 0.554" rpy="0 0 0" />
     <parent link="quori/upper_torso" />
@@ -224,5 +224,5 @@
     </visual>
   </link>
-  <joint name="head_Camera_joint" type="fixed">
+  <joint name="camera_pitch" type="fixed">
     <origin xyz="0.055 0 0.21" rpy="0 0 0" />
     <parent link="quori/head" />
@@ -243,5 +243,5 @@
     </visual>
   </link>
-  <joint name="head_Mic_joint" type="fixed">
+  <joint name="mic_array" type="fixed">
     <origin xyz="-0.008 0 0.218" rpy="0 -.3 0" />
     <parent link="quori/head" />

File: src/quori_description/urdf/ramsis_kinematics.xacro (robot description, xacro)
@@ -62,5 +62,5 @@
   <link name="ramsis/wheel_axle">
   </link>
-  <joint name="base_left" type="continuous">
+  <joint name="l_wheel" type="continuous">
     <origin xyz="0 0.12284075 0" rpy="0 0 0"/>
     <parent link="ramsis/wheel_axle"/>
@@ -69,5 +69,5 @@
     <limit effort="1" velocity="0.5"/>
   </joint>
-  <joint name="base_right" type="continuous">
+  <joint name="r_wheel" type="continuous">
     <origin xyz="0 -0.12284075 0" rpy="0 0 0"/>
     <parent link="ramsis/wheel_axle"/>
@@ -76,5 +76,5 @@
     <limit effort="1" velocity="0.5"/>
   </joint>
-  <joint name="base_turret" type="continuous">
+  <joint name="turret" type="continuous">
     <origin xyz="0 0 0.2027174" rpy="0 0 0"/>
     <parent link="ramsis/base_link"/>

Commit message: Fixes to URDF

File: src/quori_description/urdf/quori_kinematics.xacro (robot description, xacro)
@@ -14,5 +14,5 @@
     </visual>
   </link>
-  <link name="quori/upper_torso">
+  <link name="quori/body_upper">
     <inertial>
       <origin xyz="0 0 -0.01" rpy="0 0 0"/>
@@ -30,9 +30,9 @@
     <origin xyz="0 0 0.34798" rpy="0 0 0"/>
     <parent link="quori/base_link"/>
-    <child link="quori/upper_torso"/>
-    <axis xyz="0 1 0" />
-    <limit lower="-0.21" upper="0.47" effort="1" velocity="1"/>
-  </joint>
-  <link name="quori/right_arm_base">
+    <child link="quori/body_upper"/>
+    <axis xyz="0 -1 0" />
+    <limit lower="-0.47123889803846897" upper="0.2111848394913139" effort="1" velocity="1"/>
+  </joint>
+  <link name="quori/r_shoulder">
     <inertial>
       <origin xyz="0 0 0" rpy="0 0 0"/>
@@ -43,10 +43,10 @@
   <joint name="r_shoulder_pitch" type="revolute">
     <origin xyz="0.015 -0.16403066 0.43021758" rpy="0 0 0"/>
-    <parent link="quori/upper_torso"/>
-    <child link="quori/right_arm_base"/>
+    <parent link="quori/body_upper"/>
+    <child link="quori/r_shoulder"/>
     <axis xyz="0 -1 0" />
     <limit lower="-2.4" upper="2.4" effort="1" velocity="1"/>
   </joint>
-  <link name="quori/right_arm_upper">
+  <link name="quori/r_arm_upper">
     <inertial>
       <origin xyz="0 0 0" rpy="0 0 0"/>
@@ -62,11 +62,11 @@
   </link>
   <joint name="r_shoulder_roll" type="revolute">
-    <origin xyz="0 0 0" rpy="0 -1.57 0"/>
-    <parent link="quori/right_arm_base"/>
-    <child link="quori/right_arm_upper"/>
-    <axis xyz="0 0 1" />
-    <limit lower="-1.1" upper="1.1" effort="1" velocity="1"/>
-  </joint>
-  <link name="quori/right_arm_upper2lower">
+    <origin xyz="0 0 0" rpy="0 0 0" />
+    <parent link="quori/r_shoulder" />
+    <child link="quori/r_arm_upper" />
+    <axis xyz="-1 0 0" />
+    <limit lower="-1.1" upper="1.1" effort="1" velocity="1" />
+  </joint>
+  <link name="quori/r_arm_upper2lower">
     <inertial>
       <origin xyz="0 0 0.3" rpy="0 0 0"/>
@@ -82,9 +82,9 @@
     </visual>
   </link>
-  <joint name="right_arm_upper2lower_j" type="fixed">
-    <parent link="quori/right_arm_upper"/>
-    <child link="quori/right_arm_upper2lower"/>
-  </joint>
-  <link name="quori/right_arm_lower">
+  <joint name="r_arm_upper2lower_j" type="fixed">
+    <parent link="quori/r_arm_upper"/>
+    <child link="quori/r_arm_upper2lower"/>
+  </joint>
+  <link name="quori/r_arm_lower">
     <inertial>
       <origin xyz="0 0 0" rpy="0 0 0"/>
@@ -95,16 +95,14 @@
       <origin rpy="1.57 0 0" xyz="0 0 0"/>
       <geometry>
-        <mesh filename="package://quori_description/meshes/0917_Lower_Arm_left.dae" />
-      </geometry>
-    </visual>
-  </link>
-  <joint name="right_arm_lower_r1" type="revolute">
-    <origin xyz="0 -0.15 0" rpy="0 1.57 0"/>
-    <parent link="quori/right_arm_upper"/>
-    <child link="quori/right_arm_lower"/>
-    <axis xyz="0 1 0" />
-    <limit lower="-3.14" upper="3.14" effort="1" velocity="1"/>
-  </joint>
-  <link name="quori/left_arm_base">
+        <mesh filename="package://quori_description/meshes/0917_Lower_Arm_right.dae" />
+      </geometry>
+    </visual>
+  </link>
+  <joint name="r_elbow_pitch" type="fixed">
+    <origin xyz="0 -0.15 0" rpy="0 0 0" />
+    <parent link="quori/r_arm_upper" />
+    <child link="quori/r_arm_lower" />
+  </joint>
+  <link name="quori/l_shoulder">
     <inertial>
       <origin xyz="0 0 0" rpy="0 0 0"/>
@@ -114,18 +112,18 @@
   </link>
   <joint name="l_shoulder_pitch" type="revolute">
-    <origin xyz="0.015 0.16403066 0.43021758" rpy="0 0 0"/>
-    <parent link="quori/upper_torso"/>
-    <child link="quori/left_arm_base"/>
-    <axis xyz="0 1 0" />
-    <limit lower="-2.4" upper="2.4" effort="1" velocity="1"/>
-  </joint>
-  <link name="quori/left_arm_upper">
-    <inertial>
-      <origin xyz="0 0 0" rpy="0 0 0"/>
-      <mass value="0.00"/>
-      <inertia ixx="0.0"  ixy="0"  ixz="0" iyy="0.0" iyz="0" izz="0.0" />
-    </inertial>
-    <visual>
-      <origin rpy="-1.57079632679 0 -3.14" xyz="0.165 0.9765 -0.137"/>
+    <origin xyz="0.015 0.16403066 0.43021758" rpy="0 0 0" />
+    <parent link="quori/upper_torso" />
+    <child link="quori/l_shoulder" />
+    <axis xyz="0 -1 0" />
+    <limit lower="-2.4" upper="2.4" effort="1" velocity="1" />
+  </joint>
+  <link name="quori/l_arm_upper">
+    <inertial>
+      <origin xyz="0 0 0" rpy="0 0 0" />
+      <mass value="0.00" />
+      <inertia ixx="0.0"  ixy="0"  ixz="0" iyy="0.0" iyz="0" izz="0.0" />
+    </inertial>
+    <visual>
+      <origin rpy="-1.57079632679 0 -3.14" xyz="0.165 0.9765 -0.137" />
       <geometry>
         <mesh filename="package://quori_description/meshes/0917_Upper_Arm+gear_left.dae"/>
@@ -134,11 +132,11 @@
   </link>
   <joint name="l_shoulder_roll" type="revolute">
-    <origin xyz="0 0 0" rpy="0 -1.57 0"/>
-    <parent link="quori/left_arm_base"/>
-    <child link="quori/left_arm_upper"/>
-    <axis xyz="0 0 -1" />
-    <limit lower="-1.1" upper="1.1" effort="1" velocity="1"/>
-  </joint>
-  <link name="quori/left_arm_upper2lower">
+    <origin xyz="0 0 0" rpy="0 0 0" />
+    <parent link="quori/l_shoulder" />
+    <child link="quori/l_arm_upper" />
+    <axis xyz="1 0 0" />
+    <limit lower="-1.1" upper="1.1" effort="1" velocity="1" />
+  </joint>
+  <link name="quori/l_arm_upper2lower">
     <inertial>
       <origin xyz="0 0 0.3" rpy="0 0 0"/>
@@ -154,9 +152,9 @@
     </visual>
   </link>
-  <joint name="left_arm_upper2lower_j" type="fixed">
-    <parent link="quori/left_arm_upper"/>
-    <child link="quori/left_arm_upper2lower"/>
-  </joint>
-  <link name="quori/left_arm_lower">
+  <joint name="l_arm_upper2lower_j" type="fixed">
+    <parent link="quori/l_arm_upper"/>
+    <child link="quori/l_arm_upper2lower"/>
+  </joint>
+  <link name="quori/l_arm_lower">
     <inertial>
       <origin xyz="0 0 0" rpy="0 0 0"/>
@@ -171,10 +169,8 @@
     </visual>
   </link>
-  <joint name="left_arm_lower_r1" type="revolute">
-    <origin xyz="0 0.15 0" rpy="0 1.57 0"/>
-    <parent link="quori/left_arm_upper"/>
-    <child link="quori/left_arm_lower"/>
-    <axis xyz="0 1 0" />
-    <limit lower="-3.142" upper="3.142" effort="1" velocity="1"/>
+  <joint name="l_elbow_pitch" type="fixed">
+    <origin xyz="0 0.15 0" rpy="0 0 0"/>
+    <parent link="quori/l_arm_upper"/>
+    <child link="quori/l_arm_lower"/>
   </joint>
   <link name="quori/head">
@@ -200,5 +196,5 @@
   <joint name="neck" type="fixed">
     <origin xyz="0 0 0.554" rpy="0 0 0" />
-    <parent link="quori/upper_torso" />
+    <parent link="quori/body_upper" />
     <child link="quori/head" />
   </joint>

Commit message: Fix URDF

File: src/quori_description/urdf/quori_kinematics.xacro (robot description, xacro)
@@ -113,5 +113,5 @@
   <joint name="l_shoulder_pitch" type="revolute">
     <origin xyz="0.015 0.16403066 0.43021758" rpy="0 0 0" />
-    <parent link="quori/upper_torso" />
+    <parent link="quori/body_upper" />
     <child link="quori/l_shoulder" />
     <axis xyz="0 -1 0" />

Commit message: URDF working

File: src/quori_description/urdf/quori_kinematics.xacro (robot description, xacro)
@@ -93,5 +93,5 @@
     </inertial>
     <visual>
-      <origin rpy="1.57 0 0" xyz="0 0 0"/>
+      <origin rpy="1.570759635 1.570759635 0" xyz="0 0 0"/>
       <geometry>
         <mesh filename="package://quori_description/meshes/0917_Lower_Arm_right.dae" />
@@ -163,5 +163,5 @@
     </inertial>
     <visual>
-      <origin rpy="-1.57 3.14 0" xyz="0 0 0" />
+      <origin rpy="-1.570759635 -1.570759635 0" xyz="0 0 0" />
       <geometry>
         <mesh filename="package://quori_description/meshes/0917_Lower_Arm_left.dae" />
@@ -200,5 +200,5 @@
   </joint>
   <joint name="head_camera_optical_joint" type="fixed">
-    <origin xyz="0 0 0" rpy="-1.57079 0 -1.57079" />
+    <origin xyz="0 0 0" rpy="-1.57079632679 0 -1.57079632679" />
     <parent link="quori/head_camera" />
     <child link="quori/head_camera_optical" />

Commit message: Added face plugin files, need to troubleshoot why not appearing

File: src/quori_description/urdf/quori_kinematics.xacro (robot description, xacro)
@@ -185,5 +185,9 @@
         <sphere radius="0.11" />
       </geometry>
-      <material name="white"/>
+      <!-- <material name="white"/> -->
+      <plugin name="faceplugin" filename="libfaceplugin.so">
+        <height>120</height>
+        <width>240</width>
+      </plugin>
     </visual>
     <visual>
